File: Hardware/Production/MicroMod_Asset_Tracker-Panel.brd (EAGLE design)
At the start: 166.6 x 202.7 mm, 1346 parts, among them IC1 SN74AVC4T774PW, IC10 SN74AVC4T774PW, IC11 SN74AVC4T774PW, IC12 SN74AVC4T774PW, IC2 SN74AVC4T774PW, IC3 SN74AVC4T774PW, IC4 SN74AVC4T774PW, IC5 SN74AVC4T774PW, IC6 SN74AVC4T774PW, IC7 SN74AVC4T774PW, IC8 SN74AVC4T774PW, IC9 SN74AVC4T774PW, J11 microSD, J13 TP, J17 NANO_SIM, J18 SARA_USB, J19 NI, J2 JTAG, J20 JTAG, J21 SPI, J24 microSD, J26 MICROMOD-2222-C, J27 !RST!, J28 QWIIC_RIGHT_ANGLE, J32 NANO_SIM, J33 SARA_USB, J34 DIAG, J35 TP, J36 NI, J38 JTAG, J39 SPI, J4 MICROMOD-2222-C, J42 microSD, J44 MICROMOD-2222-C, J45 !RST!, J46 QWIIC_RIGHT_ANGLE, J5 SPI, J50 NANO_SIM, J51 SARA_USB, J52 DIAG, J53 TP, J54 NI, J56 JTAG, J57 SPI, J6 DIAG, J60 microSD, J62 MICROMOD-2222-C, J63 !RST!, J64 QWIIC_RIGHT_ANGLE, J68 NANO_SIM, J69 SARA_USB, J7 QWIIC_RIGHT_ANGLE, J70 DIAG, J71 TP, J72 NI, J9 !RST!, Q1 310mA/60V/1.6Ω, Q10 20V/0.2A/8MHz/1.2Ω/1Vth, Q11 310mA/60V/1.6Ω, Q12 20V/0.2A/8MHz/1.2Ω/1Vth, Q13 20V/4.2A/52mΩ/1.4W, Q14 310mA/60V/1.6Ω, Q15 310mA/60V/1.6Ω, Q16 310mA/60V/1.6Ω, Q17 20V/0.2A/8MHz/1.2Ω/1Vth, Q18 310mA/60V/1.6Ω, Q19 310mA/60V/1.6Ω, Q2 310mA/60V/1.6Ω, Q20 20V/0.2A/8MHz/1.2Ω/1Vth, Q21 20V/4.2A/52mΩ/1.4W, Q22 310mA/60V/1.6Ω, Q23 310mA/60V/1.6Ω, Q24 310mA/60V/1.6Ω, Q25 20V/0.2A/8MHz/1.2Ω/1Vth, Q26 310mA/60V/1.6Ω, Q27 310mA/60V/1.6Ω, Q28 20V/0.2A/8MHz/1.2Ω/1Vth, Q29 20V/4.2A/52mΩ/1.4W, Q3 310mA/60V/1.6Ω, Q30 310mA/60V/1.6Ω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

Commit message: v11
Parts:
- removed D53: BLUE, SparkFun-LED:LED-0603
- removed D54: 3.3V, SparkFun-DiscreteSemi:SOD-323
- removed D55: WHITE, SparkFun-LED:LED-0603
- removed D56: 1A/15V/220mV, SparkFun-DiscreteSemi:DO-214BA
- removed JP77, JP78, JP79: JUMPER-SMT_2_NC_TRACE_SILK, SparkFun-Jumpers:SMT-JUMPER_2_NC_TRACE_SILK
- removed JP80: JUMPER-SMT_2_NO_SILK, SparkFun-Jumpers:SMT-JUMPER_2_NO_SILK
- removed U$521: (no value), output:#G5#0
- removed U$522, U$523: (no value), output:#D0#1
- removed U$524: (no value), output:NANO0
- removed U$525: (no value), output:SIM0
- removed U$526, U$527: (no value), output:#SARA_#ON##0
- removed U$528: MAX17048, SparkFun-IC-Power:DFN-8
- added Q33, Q36, Q37, Q38, Q39, Q40: 310mA/60V/1.6Ω, SparkFun-DiscreteSemi:SOT323
- added Q34: 20V/0.2A/8MHz/1.2Ω/1Vth, SparkFun-DiscreteSemi:SOT-416FL
- added Q35: 20V/4.2A/52mΩ/1.4W, SparkFun-DiscreteSemi:SOT23-3
- added R181, R183: 1k, SparkFun-Resistors:0603
- added R182, R184: 100k, SparkFun-Resistors:0603
- added VIN/1, VIN/2, VIN/3, VIN/4: JUMPER-SMT_2_NC_TRACE_SILK, SparkFun-Jumpers:SMT-JUMPER_2_NC_TRACE_SILK
- D15: value 3A/10V/280mV -> 3.3V
- D16: value 3.3V -> RED; device SparkFun-DiscreteSemi:SOD-323 -> SparkFun-LED:LED-0603
- D17: value RED -> BAS70-05; device SparkFun-LED:LED-0603 -> SparkFun-DiscreteSemi:SOT23-3
- D18, D32: value BAS70-05 -> Yellow; device SparkFun-DiscreteSemi:SOT23-3 -> SparkFun-LED:LED-0603
- D20, D33: value Yellow -> DT1042-04SO-7; device SparkFun-LED:LED-0603 -> ublox:SOT23-6L
- D21, D35: value DT1042-04SO-7 -> PESD0402; device ublox:SOT23-6L -> New_Parts:0402
- D23, D36: value PESD0402 -> GREEN; device New_Parts:0402 -> SparkFun-LED:LED-0603
- D24: value GREEN -> BLUE
- D25: value BLUE -> WHITE
- D26: value 3.3V -> 1A/15V/220mV; device SparkFun-DiscreteSemi:SOD-323 -> SparkFun-DiscreteSemi:DO-214BA
- D27: value WHITE -> 3A/10V/280mV; device SparkFun-LED:LED-0603 -> SparkFun-DiscreteSemi:SOD-323
- D28: value 1A/15V/220mV -> 3.3V; device SparkFun-DiscreteSemi:DO-214BA -> SparkFun-DiscreteSemi:SOD-323
- D29: value 3A/10V/280mV -> RED; device SparkFun-DiscreteSemi:SOD-323 -> SparkFun-LED:LED-0603
- D30: value 3.3V -> BAS70-05; device SparkFun-DiscreteSemi:SOD-323 -> SparkFun-DiscreteSemi:SOT23-3
- D31, D45: value RED -> Yellow
- D34, D47, D48: value Yellow -> PESD0402; device SparkFun-LED:LED-0603 -> New_Parts:0402
- D37, D50: value PESD0402 -> BLUE; device New_Parts:0402 -> SparkFun-LED:LED-0603
- D38: value GREEN -> WHITE
- D39: value BLUE -> 1A/15V/220mV; device SparkFun-LED:LED-0603 -> SparkFun-DiscreteSemi:DO-214BA
- D40, D9: value 3.3V -> 3A/10V/280mV
- D41: value WHITE -> 3.3V; device SparkFun-LED:LED-0603 -> SparkFun-DiscreteSemi:SOD-323
- D42: value 1A/15V/220mV -> RED; device SparkFun-DiscreteSemi:DO-214BA -> SparkFun-LED:LED-0603
- D43: value 3A/10V/280mV -> BAS70-05; device SparkFun-DiscreteSemi:SOD-323 -> SparkFun-DiscreteSemi:SOT23-3
- D44: value 3.3V -> Yellow; device SparkFun-DiscreteSemi:SOD-323 -> SparkFun-LED:LED-0603
- D46: value BAS70-05 -> DT1042-04SO-7; device SparkFun-DiscreteSemi:SOT23-3 -> ublox:SOT23-6L
- D49: value DT1042-04SO-7 -> GREEN; device ublox:SOT23-6L -> SparkFun-LED:LED-0603
- D51: value PESD0402 -> WHITE; device New_Parts:0402 -> SparkFun-LED:LED-0603
- D52: value GREEN -> 1A/15V/220mV; device SparkFun-LED:LED-0603 -> SparkFun-DiscreteSemi:DO-214BA
- E11, E12, E3, E4, E5, E6, E8, E9: device New_Parts:SMA-EDGE-SMD -> SparkFun-RF:SMA-EDGE-SMD
- JP13, JP14, JP15, JP16, JP17, JP26, JP31, JP32, JP33, JP34, JP35, JP46, JP50, JP51, JP52, JP53, JP54, JP69, JP70, JP71, JP72, JP73: value JUMPER-SMT_2_NC_TRACE_SILK -> JUMPER-SMT_2_NO_SILK; device SparkFun-Jumpers:SMT-JUMPER_2_NC_TRACE_SILK -> SparkFun-Jumpers:SMT-JUMPER_2_NO_SILK
- JP19, JP39, JP58, JP59: value JUMPER-SMT_2_NC_TRACE_SILK -> (none); device SparkFun-Jumpers:SMT-JUMPER_2_NC_TRACE_SILK -> SparkFun-Jumpers:SMT-JUMPER_3_2-NC_TRACE_SILK
- JP21, JP40: value JUMPER-SMT_2_NO_SILK -> (none); device SparkFun-Jumpers:SMT-JUMPER_2_NO_SILK -> SparkFun-Jumpers:SMT-JUMPER_3_2-NC_TRACE_SILK
- JP22, JP41, JP42, JP61, JP62: value (none) -> JUMPER-SMT_2_NO_SILK; device SparkFun-Jumpers:SMT-JUMPER_3_2-NC_TRACE_SILK -> SparkFun-Jumpers:SMT-JUMPER_2_NO_SILK
- JP25, JP28, JP44, JP47, JP48, JP63, JP67, JP68: value JUMPER-SMT_2_NO_SILK -> JUMPER-SMT_2_NC_TRACE_SILK; device SparkFun-Jumpers:SMT-JUMPER_2_NO_SILK -> SparkFun-Jumpers:SMT-JUMPER_2_NC_TRACE_SILK
- JP9: value (none) -> JUMPER-SMT_2_NC_TRACE_SILK; device SparkFun-Jumpers:SMT-JUMPER_3_2-NC_TRACE_SILK -> SparkFun-Jumpers:SMT-JUMPER_2_NC_TRACE_SILK
- Q11, Q14, Q24, Q31: value 310mA/60V/1.6Ω -> 20V/0.2A/8MHz/1.2Ω/1Vth; device SparkFun-DiscreteSemi:SOT323 -> SparkFun-DiscreteSemi:SOT-416FL
- Q12, Q17, Q20, Q28, Q8: value 20V/0.2A/8MHz/1.2Ω/1Vth -> 310mA/60V/1.6Ω; device SparkFun-DiscreteSemi:SOT-416FL -> SparkFun-DiscreteSemi:SOT323
- Q13, Q29: value 20V/4.2A/52mΩ/1.4W -> 310mA/60V/1.6Ω; device SparkFun-DiscreteSemi:SOT23-3 -> SparkFun-DiscreteSemi:SOT323
- Q15: value 310mA/60V/1.6Ω -> 20V/4.2A/52mΩ/1.4W; device SparkFun-DiscreteSemi:SOT323 -> SparkFun-DiscreteSemi:SOT23-3
- Q21: value 20V/4.2A/52mΩ/1.4W -> 20V/0.2A/8MHz/1.2Ω/1Vth; device SparkFun-DiscreteSemi:SOT23-3 -> SparkFun-DiscreteSemi:SOT-416FL
- Q25: value 20V/0.2A/8MHz/1.2Ω/1Vth -> 20V/4.2A/52mΩ/1.4W; device SparkFun-DiscreteSemi:SOT-416FL -> SparkFun-DiscreteSemi:SOT23-3
- R100: value 4.7k -> 100k
- R101, R108, R115, R147, R160, R161: value 2.2k -> 1k
- R102, R56: value 2.2k -> 4.7k
- R103, R104, R143, R149, R58: value 100k -> 2.2k
- R105, R146, R151: value 2.2k -> 100k
- R107, R152, R163: value 1k -> 2.2k
- R109, R51, R96: value 10k -> 2.2k
- R110: value 10 -> 10k
- R111: value 100k -> 10
- R112: value 200k -> 100k
- R113, R159: value 1k -> 200k
- R117, R162: value 0 -> 2.2k
- R118: value 1k -> 0
- R119: value 470 -> 1k
- R120, R166: value 1k -> 100
- R122, R168: value 0 -> 470
- R124, R169, R170: value 100k -> 0
- R13, R135, R180: value 100k -> 1k
- R133, R158, R178, R179, R54: value 1k -> 100k
- R136, R45, R92: value 5.1k -> 100k
- R137, R91: value 5.1k -> 1k
- R138: value 3.3k -> 100k
- R139, R140, R94: value 2.2k -> 5.1k
- R141: value 10k -> 3.3k
- R142, R97: value 20k -> 2.2k
- R144: value 1k -> 10k
- R145: value 4.7k -> 20k
- R148: value 100k -> 4.7k
- R154: value 10k -> 1k
- R155: value 10 -> 2.2k
- R156, R98: value 100k -> 10k
- R157: value 200k -> 10
- R164: value 470 -> 0
- R167: value 0 -> 1k
- R33, R74: value 470 -> 100
- R35, R76: value 1k -> 470
- R47, R93: value 3.3k -> 5.1k
- R49, R95: value 2.2k -> 3.3k
- R52: value 20k -> 10k
- R53: value 100k -> 20k
- R55: value 4.7k -> 1k
- R99: value 1k -> 20k
- U$110: device output:#ANT_PWR#0 -> output:#SARA_#ON##0
- U$118, U$119, U$262: device output:#SARA_#ON##0 -> SparkFun-MicroMod:MICROMOD_LOGO_.35
- U$120: device output:#G10#0 -> output:#CIPO#2
- U$121: device output:#G9#0 -> output:#CIPO#2
- U$133: device SparkFun-MicroMod:MICROMOD_LOGO_.35 -> output:#VIN#3#0
- U$134: device SparkFun-MicroMod:MICROMOD_LOGO_.35 -> output:#ICM_INT#0
- U$135, U$136: device output:#CIPO#2 -> output:#COPI#1
- U$137, U$138, U$401, U$402: device output:#COPI#1 -> output:#GND#4
- U$139, U$140: device output:#GND#4 -> output:#SCK#0
- U$141, U$142: device output:#SCK#0 -> output:#GND#4
- U$143, U$144, U$403, U$404: device output:#GND#4 -> output:#A0#5
- U$145, U$146: device output:#A0#5 -> output:#A1#4
- U$147, U$148: device output:#A1#4 -> output:#D0#1
- U$149, U$150: device output:#D0#1 -> output:#D1#0
- U$151, U$152: device output:#D1#0 -> output:#PWM0#3
- U$153, U$154: device output:#PWM0#3 -> output:#PWM1#2
- U$155, U$156: device output:#PWM1#2 -> output:#3V3#1
- U$157, U$158, U$180, U$181: device output:#3V3#1 -> output:#GND#0
- U$159, U$160, U$182, U$183: device output:#GND#0 -> output:#SCL#3
- U$161, U$162, U$184, U$185: device output:#SCL#3 -> output:#SDA#2
- U$163: device output:#SDA#2 -> output:3V37
- U$164: device output:#SDA#2 -> output:BOOT5
- U$165: device output:3V37 -> output:RESET6
- U$166: device output:BOOT5 -> output:VIN8
- U$167: device output:RESET6 -> output:X1
- U$168: device output:VIN8 -> output:Y2
- U$169: device output:X1 -> output:Z0
- U$170: device output:Y2 -> output:#MEAS#2
- U$171: device output:Z0 -> output:SWD0
- U$172: device output:#MEAS#2 -> output:#BYP#1
- U$173: device output:SWD0 -> output:#RST#1
- U$174: device output:#BYP#1 -> output:#VE#0
- U$175: device output:#RST#1 -> output:#3V3#0
- U$176: device output:#VE#0 -> output:#VIN#1
- U$177: device output:#3V3#0 -> output:MICROSD0
- U$178: device output:#VIN#1 -> output:#3V3#1
- U$179: device output:MICROSD0 -> output:#3V3#1
- U$186: device output:#SDA#2 -> output:#I�C#0
- U$187, U$428: device output:#SDA#2 -> output:Y2
- U$188: device output:#I�C#0 -> output:X1
- U$189: device output:Y2 -> output:Z0
- U$190: device output:X1 -> output:#GND#4
- U$191: device output:Z0 -> output:#GND#4
- U$192, U$193: device output:#GND#4 -> output:#TP#0
- U$194, U$195: device output:#TP#0 -> output:#NI#0
- U$196, U$197, U$328, U$329: device output:#NI#0 -> output:#SARA_USB_D##0
- U$200, U$201, U$330, U$331: device output:#SARA_USB_D##0 -> output:#SARA_USB_DET#0
- U$202, U$203: device output:#SARA_USB_DET#0 -> output:#VIN#0
- U$204, U$205: device output:#VIN#0 -> output:#3#3V#0
- U$206, U$207: device output:#3#3V#0 -> output:#VCCIO#0
- U$208, U$209: device output:#VCCIO#0 -> output:#1#8V#0
- U$210: device output:#1#8V#0 -> output:#RST#1
- U$211: device output:#1#8V#0 -> output:#MEAS#2
- U$212: device output:#RST#1 -> output:NI0
- U$213: device output:#MEAS#2 -> output:TP0
- U$214: device output:NI0 -> output:#USB_D##0
- U$215: device output:TP0 -> output:#USB_D##0
- U$216: device output:#USB_D##0 -> output:#V_USB#0
- U$217: device output:#USB_D##0 -> output:AG0
- U$218: device output:#V_USB#0 -> output:M0
- U$219: device output:AG0 -> output:CHARGE0
- U$220: device output:M0 -> output:ASSET_TRACKER0
- U$221: device output:CHARGE0 -> output:MIC0
- U$222: device output:ASSET_TRACKER0 -> output:#EN#0
- U$223: device output:MIC0 -> output:#SARA_I�C#0
- U$224: device output:#EN#0 -> output:#SARA_I�C#0
- U$225, U$226: device output:#SARA_I�C#0 -> output:LTE0
- U$227, U$228: device output:LTE0 -> output:GNSS0
- U$229: device output:GNSS0 -> output:#SARA_INT#0
- U$230: device output:GNSS0 -> output:#RI#0
- U$231: device output:#SARA_INT#0 -> output:#DSR#0
- U$232: device output:#RI#0 -> output:#SD_#CS##0
- U$233: device output:#DSR#0 -> output:#IMU_PWR#0
- U$234: device output:#SD_#CS##0 -> output:#LTE_PWR#0
- U$235: device output:#IMU_PWR#0 -> output:#SD_PWR#0
- U$236: device output:#LTE_PWR#0 -> output:#SARA_SCL#0
- U$237: device output:#SD_PWR#0 -> output:#SARA_SDA#0
- U$238: device output:#ANT_PWR#0 -> output:#CIPO#0
- U$239: device output:#SARA_SCL#0 -> output:22220
- U$240: device output:#SARA_SDA#0 -> output:SARA_ON0
- U$241: device output:#CIPO#0 -> output:ON0
- U$242: device output:22220 -> output:#PDM_CLK#0
- U$243: device output:SARA_ON0 -> output:#PDM_DAT#0
- U$244: device output:ON0 -> output:#DSR#0
- U$245: device output:#PDM_CLK#0 -> output:#G0#0
- U$246: device output:#PDM_DAT#0 -> output:#G1#0
- U$247: device output:#DSR#0 -> output:#G2#0
- U$248: device output:#G10#0 -> output:#G3#0
- U$249: device output:#G9#0 -> output:#G4#0
- U$250: device output:#G0#0 -> output:#G7#0
- U$251: device output:#G1#0 -> output:#G6#0
- U$252: device output:#G2#0 -> output:#G5#0
- U$253: device output:#G3#0 -> output:#D0#1
- U$254: device output:#G4#0 -> output:#D0#1
- U$255: device output:#G7#0 -> output:NANO0
- U$256: device output:#G6#0 -> output:SIM0
- U$257: value (none) -> MAX17048; device output:#G5#0 -> SparkFun-IC-Power:DFN-8
- U$258: device output:#D0#1 -> output:#VIN#3#0
- U$259: device output:#D0#1 -> output:#ICM_INT#0
- U$260: device output:NANO0 -> output:#SARA_#ON##0
- U$261: device output:SIM0 -> SparkFun-MicroMod:MICROMOD_LOGO_.35
- U$263, U$394: device output:#SARA_#ON##0 -> output:#CIPO#2
- U$264: value MAX17048 -> (none); device SparkFun-IC-Power:DFN-8 -> output:#CIPO#2
- U$265, U$266: device SparkFun-MicroMod:MICROMOD_LOGO_.35 -> output:#COPI#1
- U$267, U$268: device output:#CIPO#2 -> output:#GND#4
- U$269, U$270: device output:#COPI#1 -> output:#SCK#0
- U$273, U$274: device output:#SCK#0 -> output:#A0#5
- U$275, U$276: device output:#GND#4 -> output:#A1#4
- U$277, U$278: device output:#A0#5 -> output:#D0#1
- U$279, U$280: device output:#A1#4 -> output:#D1#0
- U$281, U$282: device output:#D0#1 -> output:#PWM0#3
- U$283, U$284: device output:#D1#0 -> output:#PWM1#2
- U$285, U$286: device output:#PWM0#3 -> output:#3V3#1
- U$287, U$288: device output:#PWM1#2 -> output:#GND#0
- U$289, U$290, U$312, U$313: device output:#3V3#1 -> output:#SCL#3
- U$291, U$292, U$314, U$315: device output:#GND#0 -> output:#SDA#2
- U$293: device output:#SCL#3 -> output:3V37
- U$294: device output:#SCL#3 -> output:BOOT5
- U$295: device output:#SDA#2 -> output:RESET6
- U$296: device output:#SDA#2 -> output:VIN8
- U$297: device output:3V37 -> output:X1
- U$298: device output:BOOT5 -> output:Y2
- U$299: device output:RESET6 -> output:Z0
- U$300: device output:VIN8 -> output:#MEAS#2
- U$301: device output:X1 -> output:SWD0
- U$302: device output:Y2 -> output:#BYP#1
- U$303: device output:Z0 -> output:#RST#1
- U$304: device output:#MEAS#2 -> output:#VE#0
- U$305: device output:SWD0 -> output:#3V3#0
- U$306: device output:#BYP#1 -> output:#VIN#1
- U$307: device output:#RST#1 -> output:MICROSD0
- U$308: device output:#VE#0 -> output:#3V3#1
- U$309: device output:#3V3#0 -> output:#3V3#1
- U$310: device output:#VIN#1 -> output:#GND#0
- U$311: device output:MICROSD0 -> output:#GND#0
- U$316: device output:#SCL#3 -> output:#I�C#0
- U$317: device output:#SCL#3 -> output:Y2
- U$318, U$427: device output:#SDA#2 -> output:X1
- U$319: device output:#SDA#2 -> output:Z0
- U$320: device output:#I�C#0 -> output:#GND#4
- U$321: device output:Y2 -> output:#GND#4
- U$322: device output:X1 -> output:#TP#0
- U$323: device output:Z0 -> output:#TP#0
- U$324, U$325: device output:#GND#4 -> output:#NI#0
- U$326, U$327, U$458, U$459: device output:#TP#0 -> output:#SARA_USB_D##0
- U$332, U$333, U$462, U$463: device output:#SARA_USB_D##0 -> output:#VIN#0
- U$334, U$335: device output:#SARA_USB_DET#0 -> output:#3#3V#0
- U$336, U$337: device output:#VIN#0 -> output:#VCCIO#0
- U$338, U$339: device output:#3#3V#0 -> output:#1#8V#0
- U$340: device output:#VCCIO#0 -> output:#RST#1
- U$341: device output:#VCCIO#0 -> output:#MEAS#2
- U$342: device output:#1#8V#0 -> output:NI0
- U$343: device output:#1#8V#0 -> output:TP0
- U$344: device output:#RST#1 -> output:#USB_D##0
- U$345: device output:#MEAS#2 -> output:#USB_D##0
- U$346: device output:NI0 -> output:#V_USB#0
- U$347: device output:TP0 -> output:AG0
- U$348: device output:#USB_D##0 -> output:M0
- U$349: device output:#USB_D##0 -> output:CHARGE0
- U$350: device output:#V_USB#0 -> output:ASSET_TRACKER0
- U$351: device output:AG0 -> output:MIC0
- U$352: device output:M0 -> output:#EN#0
- U$353: device output:CHARGE0 -> output:#SARA_I�C#0
- U$354: device output:ASSET_TRACKER0 -> output:#SARA_I�C#0
- U$355: device output:MIC0 -> output:LTE0
- U$356: device output:#EN#0 -> output:LTE0
- U$357, U$358: device output:#SARA_I�C#0 -> output:GNSS0
- U$359: device output:LTE0 -> output:#SARA_INT#0
- U$360: device output:LTE0 -> output:#RI#0
- U$361: device output:GNSS0 -> output:#DSR#0
- U$362: device output:GNSS0 -> output:#SD_#CS##0
- U$363: device output:#SARA_INT#0 -> output:#IMU_PWR#0
- U$364: device output:#RI#0 -> output:#LTE_PWR#0
- U$365: device output:#DSR#0 -> output:#SD_PWR#0
- U$366: device output:#SD_#CS##0 -> output:#SARA_SCL#0
- U$367: device output:#IMU_PWR#0 -> output:#SARA_SDA#0
- U$368: device output:#LTE_PWR#0 -> output:#CIPO#0
- U$369: device output:#SD_PWR#0 -> output:22220
- U$370: device output:#ANT_PWR#0 -> output:SARA_ON0
- U$371: device output:#SARA_SCL#0 -> output:ON0
- U$372: device output:#SARA_SDA#0 -> output:#PDM_CLK#0
- U$373: device output:#CIPO#0 -> output:#PDM_DAT#0
- U$374: device output:22220 -> output:#DSR#0
- U$375: device output:SARA_ON0 -> output:#G0#0
- U$376: device output:ON0 -> output:#G1#0
- U$377: device output:#PDM_CLK#0 -> output:#G2#0
- U$378: device output:#PDM_DAT#0 -> output:#G3#0
- U$379: device output:#DSR#0 -> output:#G4#0
- U$380: device output:#G10#0 -> output:#G7#0
- U$381: device output:#G9#0 -> output:#G6#0
- U$382: device output:#G0#0 -> output:#G5#0
- U$383: device output:#G1#0 -> output:#D0#1
- U$384: device output:#G2#0 -> output:#D0#1
- U$385: device output:#G3#0 -> output:NANO0
- U$386: device output:#G4#0 -> output:SIM0
- U$387: value (none) -> MAX17048; device output:#G7#0 -> SparkFun-IC-Power:DFN-8
- U$388: device output:#G6#0 -> output:#VIN#3#0
- U$389: device output:#G5#0 -> output:#ICM_INT#0
- U$390: device output:#D0#1 -> output:#SARA_#ON##0
- U$391: device output:#D0#1 -> SparkFun-MicroMod:MICROMOD_LOGO_.35
- U$392: device output:NANO0 -> SparkFun-MicroMod:MICROMOD_LOGO_.35
- U$393: device output:SIM0 -> output:#CIPO#2
- U$395: device output:#SARA_#ON##0 -> output:#COPI#1
- U$396: value MAX17048 -> (none); device SparkFun-IC-Power:DFN-8 -> output:#COPI#1
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Connections:
- removed net G32: J62.44, JP71.1
- removed net G33: J62.46, JP72.1
- removed net G34: J62.48, JP73.1
- removed net G35: J62.73, JP74.1
- removed net G36: J62.71, JP75.1
- removed net G37: J62.69, JP76.1
- removed net G38: J62.63, JP79.1
- removed net G39: J62.65, JP80.1
- removed net N$104 (its old number): Q18.1, R113.2
- removed net N$107 (its old number): JP46.1, R108.2
- removed net N$131 (its old number): D45.A, R144.1
- removed net N$141 (its old number): C114.1, D50.1, L7.P$1, R154.2
- removed net N$149 (its old number): R162.2, U26.4
- removed net N$152 (its old number): D52.C, R164.2
- removed net N$48 (its old number): D19.A, R55.1
- removed net N$59 (its old number): C50.1, D22.1, L3.P$1, R64.2
- removed net N$64 (its old number): Q11.1, R69.2
- removed net N$66 (its old number): JP26.1, R63.2
- removed net N$69 (its old number): J35.1, Q14.3, R74.1, R79.1
- removed net N$71 (its old number): Q15.1, R75.2
- removed net N$78 (its old number): Q16.1, R88.2
- removed net N$79 (its old number): J26.52, JP38.1
- removed net N$86 (its old number): JP41.3, R95.2
- new net ANT_REG_EN: Q9.3, R45.2, U3.3
- new net ANT_REG_EN1: Q20.3, R92.2, U12.3
- new net ANT_REG_EN2: Q30.3, R138.2, U22.3
- new net ANT_REG_EN3: Q40.3, R184.2, U30.3
- new net N$123: R123.2, U18.13
- new net N$129: J44.50, JP55.1
- new net N$137: J55.B5, R140.2
- new net N$140: JP58.1, R142.2
- new net N$164: D49.C, R166.2
- new net N$165: Q37.1, R167.2
- new net N$166: J72.1, Q37.3, R168.1, R172.1
- new net N$167: D50.C, R168.2
- new net N$168: R169.2, U26.13
- new net N$169: R170.2, U26.12
- new net N$170: J62.53, JP64.2
- new net N$171: J62.51, JP65.2
- new net N$172: Q38.1, R180.2
- new net N$173: J62.52, JP75.1
- new net N$174: J62.50, JP74.1
- new net N$175: D51.C, R181.2
- new net N$177: R145.2, VIN/4.1
- new net N$178: J62.16, JP76.2
- new net N$179: Q39.1, R183.2
- new net N$180: Q39.3, Q40.1, R158.2
- new net N$43: J3.B5, R47.2
- new net N$55: D18.A, R56.1
- new net N$56: D15.C, R54.1, U4.5, VE1.2
- new net N$58: JP21.1, R57.2
- new net N$61: D19.C, R62.2
- new net N$67: Q12.1, R68.2
- new net N$74: D23.C, R74.2
- new net N$75: Q17.1, R75.2
- new net N$82: Q18.1, R88.2
- new net N$88: J26.16, JP38.2
- new net N$99: R102.2, VIN_LED2.1
- net !BOOT!: no longer R13.1
- net !BOOT!1: no longer R59.1
- net !BOOT!2: no longer R104.1
- net !BOOT!3: no longer R149.1
- net !RESET!1: now also R59.1; no longer R58.1
- net !RESET!2: now also R105.1; no longer R103.1
- net !RESET!3: now also R151.1; no longer R148.1
- net 1.8V1: now also Q11.1; no longer Q8.1
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Routing:
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Other:
- board text added: "v11"
- board text removed: "v10"

Commit message: Adding production files for v11
Parts:
- removed TP93, TP94, TP95, TP96: TEST-POINT3, SparkFun-Connectors:PAD.03X.03
- added JP77, JP78, JP79: JUMPER-SMT_2_NC_TRACE_SILK, SparkFun-Jumpers:SMT-JUMPER_2_NC_TRACE_SILK
- added JP80: JUMPER-SMT_3_1-NC_TRACE_SILK, SparkFun-Jumpers:SMT-JUMPER_3_1-NC_TRACE_SILK
- added U$521: (no value), output:#ICM_INT#0
- added U$522: (no value), output:#SARA_#ON##0
- added U$523: (no value), output:#EXT_INT#0
- added U$524: (no value), output:#GPIO3#0
- added U33: 3.3V, SparkFun-IC-Power:SOT23-5
- added U34: PCA9306, SparkFun-IC-Comms:VSSOP_8PIN
- added U35: 74HC1G04, SparkFun-IC-Logic:SOT353
- added U36: MAX17048, SparkFun-IC-Power:DFN-8
- JP19, JP40: value (none) -> JUMPER-SMT_3_1-NC_TRACE_SILK; device SparkFun-Jumpers:SMT-JUMPER_3_2-NC_TRACE_SILK -> SparkFun-Jumpers:SMT-JUMPER_3_1-NC_TRACE_SILK
- JP22, JP41, JP42, JP61, JP62: value JUMPER-SMT_2_NO_SILK -> (none); device SparkFun-Jumpers:SMT-JUMPER_2_NO_SILK -> SparkFun-Jumpers:SMT-JUMPER_3_2-NC_TRACE_SILK
- JP25, JP28, JP36, JP44, JP47, JP48, JP55, JP56, JP63, JP67, JP68, JP74, JP75, JP76: value JUMPER-SMT_2_NC_TRACE_SILK -> JUMPER-SMT_2_NO_SILK; device SparkFun-Jumpers:SMT-JUMPER_2_NC_TRACE_SILK -> SparkFun-Jumpers:SMT-JUMPER_2_NO_SILK
- JP26, JP31, JP46, JP50, JP51, JP69, JP70, JP71: value JUMPER-SMT_2_NO_SILK -> JUMPER-SMT_2_NC_TRACE_SILK; device SparkFun-Jumpers:SMT-JUMPER_2_NO_SILK -> SparkFun-Jumpers:SMT-JUMPER_2_NC_TRACE_SILK
- JP39, JP58, JP59: value (none) -> JUMPER-SMT_2_NC_TRACE_SILK; device SparkFun-Jumpers:SMT-JUMPER_3_2-NC_TRACE_SILK -> SparkFun-Jumpers:SMT-JUMPER_2_NC_TRACE_SILK
- JP60: value JUMPER-SMT_2_NO_SILK -> JUMPER-SMT_3_1-NC_TRACE_SILK; device SparkFun-Jumpers:SMT-JUMPER_2_NO_SILK -> SparkFun-Jumpers:SMT-JUMPER_3_1-NC_TRACE_SILK
- U$118, U$261, U$392: device SparkFun-MicroMod:MICROMOD_LOGO_.35 -> output:#EXT_INT#0
- U$119, U$262: device SparkFun-MicroMod:MICROMOD_LOGO_.35 -> output:#GPIO3#0
- U$120, U$121, U$263, U$264, U$394: device output:#CIPO#2 -> SparkFun-MicroMod:MICROMOD_LOGO_.35
- U$132: value MAX17048 -> (none); device SparkFun-IC-Power:DFN-8 -> output:#CIPO#2
- U$135, U$265, U$266, U$396: device output:#COPI#1 -> output:#CIPO#2
- U$137, U$267, U$268, U$398: device output:#GND#4 -> output:#COPI#1
- U$139, U$269, U$270, U$400: device output:#SCK#0 -> output:#GND#4
- U$141, U$271, U$272, U$402: device output:#GND#4 -> output:#SCK#0
- U$143, U$273, U$274, U$404: device output:#A0#5 -> output:#GND#4
- U$145, U$275, U$276, U$406: device output:#A1#4 -> output:#A0#5
- U$147, U$277, U$278, U$408: device output:#D0#1 -> output:#A1#4
- U$149, U$279, U$280, U$410: device output:#D1#0 -> output:#D0#1
- U$151, U$281, U$282, U$412: device output:#PWM0#3 -> output:#D1#0
- U$153, U$283, U$284, U$414: device output:#PWM1#2 -> output:#PWM0#3
- U$155, U$285, U$286, U$416: device output:#3V3#1 -> output:#PWM1#2
- U$157, U$180, U$287, U$288, U$310, U$311, U$418, U$441: device output:#GND#0 -> output:#3V3#1
- U$159, U$182, U$289, U$290, U$312, U$313, U$420, U$443: device output:#SCL#3 -> output:#GND#0
- U$161, U$184, U$291, U$292, U$314, U$315, U$422, U$445: device output:#SDA#2 -> output:#SCL#3
- U$163, U$293: device output:3V37 -> output:#SDA#2
- U$164: device output:BOOT5 -> output:3V37
- U$165: device output:RESET6 -> output:BOOT5
- U$166: device output:VIN8 -> output:RESET6
- U$167: device output:X1 -> output:VIN8
- U$168: device output:Y2 -> output:X1
- U$169, U$319: device output:Z0 -> output:Y2
- U$170: device output:#MEAS#2 -> output:Z0
- U$171: device output:SWD0 -> output:#MEAS#2
- U$172: device output:#BYP#1 -> output:SWD0
- U$173: device output:#RST#1 -> output:#BYP#1
- U$174: device output:#VE#0 -> output:#RST#1
- U$175: device output:#3V3#0 -> output:#VE#0
- U$176: device output:#VIN#1 -> output:#3V3#0
- U$177: device output:MICROSD0 -> output:#VIN#1
- U$178, U$309: device output:#3V3#1 -> output:MICROSD0
- U$186, U$316: device output:#I�C#0 -> output:#SDA#2
- U$187: device output:Y2 -> output:#I�C#0
- U$188: device output:X1 -> output:Y2
- U$189, U$299: device output:Z0 -> output:X1
- U$190, U$321: device output:#GND#4 -> output:Z0
- U$192, U$322, U$323, U$453: device output:#TP#0 -> output:#GND#4
- U$194, U$324, U$325, U$455: device output:#NI#0 -> output:#TP#0
- U$196, U$326, U$327, U$457, U$458: device output:#SARA_USB_D##0 -> output:#NI#0
- U$200, U$330, U$331, U$460, U$461: device output:#SARA_USB_DET#0 -> output:#SARA_USB_D##0
- U$202, U$332, U$333, U$463: device output:#VIN#0 -> output:#SARA_USB_DET#0
- U$204, U$334, U$335, U$465: device output:#3#3V#0 -> output:#VIN#0
- U$206, U$336, U$337, U$467: device output:#VCCIO#0 -> output:#3#3V#0
- U$208, U$338, U$339, U$469: device output:#1#8V#0 -> output:#VCCIO#0
- U$210, U$340: device output:#RST#1 -> output:#1#8V#0
- U$211: device output:#MEAS#2 -> output:#RST#1
- U$212: device output:NI0 -> output:#MEAS#2
- U$213: device output:TP0 -> output:NI0
- U$214, U$345: device output:#USB_D##0 -> output:TP0
- U$216, U$346: device output:#V_USB#0 -> output:#USB_D##0
- U$217: device output:AG0 -> output:#V_USB#0
- U$218: device output:M0 -> output:AG0
- U$219: device output:CHARGE0 -> output:M0
- U$220: device output:ASSET_TRACKER0 -> output:CHARGE0
- U$221: device output:MIC0 -> output:ASSET_TRACKER0
- U$222: device output:#EN#0 -> output:MIC0
- U$223, U$354: device output:#SARA_I�C#0 -> output:#EN#0
- U$225, U$355, U$356, U$486: device output:LTE0 -> output:#SARA_I�C#0
- U$227, U$357, U$358, U$488: device output:GNSS0 -> output:LTE0
- U$229, U$359: device output:#SARA_INT#0 -> output:GNSS0
- U$230: device output:#RI#0 -> output:#SARA_INT#0
- U$231: device output:#DSR#0 -> output:#RI#0
- U$232: device output:#SD_#CS##0 -> output:#DSR#0
- U$233: device output:#IMU_PWR#0 -> output:#SD_#CS##0
- U$234: device output:#LTE_PWR#0 -> output:#IMU_PWR#0
- U$235: device output:#SD_PWR#0 -> output:#LTE_PWR#0
- U$236: device output:#SARA_SCL#0 -> output:#SD_PWR#0
- U$237: device output:#SARA_SDA#0 -> output:#SARA_SCL#0
- U$238: device output:#CIPO#0 -> output:#SARA_SDA#0
- U$239: device output:22220 -> output:#CIPO#0
- U$240: device output:SARA_ON0 -> output:22220
- U$241: device output:ON0 -> output:SARA_ON0
- U$242: device output:#PDM_CLK#0 -> output:ON0
- U$243: device output:#PDM_DAT#0 -> output:#PDM_CLK#0
- U$244: device output:#DSR#0 -> output:#PDM_DAT#0
- U$245: device output:#G0#0 -> output:#DSR#0
- U$246: device output:#G1#0 -> output:#G0#0
- U$247: device output:#G2#0 -> output:#G1#0
- U$248: device output:#G3#0 -> output:#G2#0
- U$249: device output:#G4#0 -> output:#G3#0
- U$250: device output:#G7#0 -> output:#G4#0
- U$251: device output:#G6#0 -> output:#G7#0
- U$252: device output:#G5#0 -> output:#G6#0
- U$253, U$384: device output:#D0#1 -> output:#G5#0
- U$255, U$385: device output:NANO0 -> output:#D0#1
- U$256: device output:SIM0 -> output:NANO0
- U$257: value MAX17048 -> (none); device SparkFun-IC-Power:DFN-8 -> output:SIM0
- U$294, U$424: device output:BOOT5 -> output:#SDA#2
- U$295: device output:RESET6 -> output:3V37
- U$296: device output:VIN8 -> output:BOOT5
- U$297: device output:X1 -> output:RESET6
- U$298: device output:Y2 -> output:VIN8
- U$300: device output:#MEAS#2 -> output:Y2
- U$301: device output:SWD0 -> output:Z0
- U$302: device output:#BYP#1 -> output:#MEAS#2
- U$303: device output:#RST#1 -> output:SWD0
- U$304: device output:#VE#0 -> output:#BYP#1
- U$305: device output:#3V3#0 -> output:#RST#1
- U$306: device output:#VIN#1 -> output:#VE#0
- U$307: device output:MICROSD0 -> output:#3V3#0
- U$308, U$439: device output:#3V3#1 -> output:#VIN#1
- U$317, U$447: device output:Y2 -> output:#SDA#2
- U$318: device output:X1 -> output:#I�C#0
- U$320, U$451: device output:#GND#4 -> output:X1
- U$341, U$471: device output:#MEAS#2 -> output:#1#8V#0
- U$342: device output:NI0 -> output:#RST#1
- U$343: device output:TP0 -> output:#MEAS#2
- U$344, U$475: device output:#USB_D##0 -> output:NI0
- U$347, U$477: device output:AG0 -> output:#USB_D##0
- U$348: device output:M0 -> output:#V_USB#0
- U$349: device output:CHARGE0 -> output:AG0
- U$350: device output:ASSET_TRACKER0 -> output:M0
- U$351: device output:MIC0 -> output:CHARGE0
- U$352: device output:#EN#0 -> output:ASSET_TRACKER0
- U$353, U$484: device output:#SARA_I�C#0 -> output:MIC0
- U$360, U$490: device output:#RI#0 -> output:GNSS0
- U$361: device output:#DSR#0 -> output:#SARA_INT#0
- U$362: device output:#SD_#CS##0 -> output:#RI#0
- U$363: device output:#IMU_PWR#0 -> output:#DSR#0
- U$364: device output:#LTE_PWR#0 -> output:#SD_#CS##0
- U$365: device output:#SD_PWR#0 -> output:#IMU_PWR#0
- U$366: device output:#SARA_SCL#0 -> output:#LTE_PWR#0
- U$367: device output:#SARA_SDA#0 -> output:#SD_PWR#0
- U$368: device output:#CIPO#0 -> output:#SARA_SCL#0
- U$369: device output:22220 -> output:#SARA_SDA#0
- U$370: device output:SARA_ON0 -> output:#CIPO#0
- U$371: device output:ON0 -> output:22220
- U$372: device output:#PDM_CLK#0 -> output:SARA_ON0
- U$373: device output:#PDM_DAT#0 -> output:ON0
- U$374: device output:#DSR#0 -> output:#PDM_CLK#0
- U$375: device output:#G0#0 -> output:#PDM_DAT#0
- U$376: device output:#G1#0 -> output:#DSR#0
- U$377: device output:#G2#0 -> output:#G0#0
- U$378: device output:#G3#0 -> output:#G1#0
- U$379: device output:#G4#0 -> output:#G2#0
- U$380: device output:#G7#0 -> output:#G3#0
- U$381: device output:#G6#0 -> output:#G4#0
- U$382: device output:#G5#0 -> output:#G7#0
- U$383, U$514: device output:#D0#1 -> output:#G6#0
- U$386, U$516: device output:SIM0 -> output:#D0#1
- U$387: value MAX17048 -> (none); device SparkFun-IC-Power:DFN-8 -> output:NANO0
- U$388: device output:#VIN#3#0 -> output:SIM0
- U$389: device output:#ICM_INT#0 -> output:#VIN#3#0
- U$390: device output:#SARA_#ON##0 -> output:#ICM_INT#0
- U$391: device SparkFun-MicroMod:MICROMOD_LOGO_.35 -> output:#SARA_#ON##0
- U$393: device output:#CIPO#2 -> output:#GPIO3#0
- U$395: device output:#COPI#1 -> SparkFun-MicroMod:MICROMOD_LOGO_.35
- U$397: device output:#GND#4 -> output:#CIPO#2
- U$399: device output:#SCK#0 -> output:#COPI#1
- U$403: device output:#A0#5 -> output:#SCK#0
- U$405: device output:#A1#4 -> output:#GND#4
- U$407: device output:#D0#1 -> output:#A0#5
- U$409: device output:#D1#0 -> output:#A1#4
- U$411: device output:#PWM0#3 -> output:#D0#1
- U$413: device output:#PWM1#2 -> output:#D1#0
- U$415: device output:#3V3#1 -> output:#PWM0#3
- U$417: device output:#GND#0 -> output:#PWM1#2
- U$419, U$442: device output:#SCL#3 -> output:#3V3#1
- U$421, U$444: device output:#SDA#2 -> output:#GND#0
- U$423: device output:3V37 -> output:#SCL#3
- U$425: device output:RESET6 -> output:#SDA#2
- U$426: device output:VIN8 -> output:3V37
- U$427: device output:X1 -> output:BOOT5
- U$428: device output:Y2 -> output:RESET6
- U$429: device output:Z0 -> output:VIN8
- U$430: device output:#MEAS#2 -> output:X1
- U$431: device output:SWD0 -> output:Y2
- U$432: device output:#BYP#1 -> output:Z0
- U$433: device output:#RST#1 -> output:#MEAS#2
- U$434: device output:#VE#0 -> output:SWD0
- U$435: device output:#3V3#0 -> output:#BYP#1
- U$436: device output:#VIN#1 -> output:#RST#1
- U$437: device output:MICROSD0 -> output:#VE#0
- U$438: device output:#3V3#1 -> output:#3V3#0
- U$440: device output:#GND#0 -> output:MICROSD0
- U$446: device output:#I�C#0 -> output:#SCL#3
- U$448: device output:X1 -> output:#SDA#2
- U$449: device output:Z0 -> output:#I�C#0
- U$450: device output:#GND#4 -> output:Y2
- U$452: device output:#TP#0 -> output:Z0
- U$454: device output:#NI#0 -> output:#GND#4
- U$456: device output:#SARA_USB_D##0 -> output:#TP#0
- U$462: device output:#VIN#0 -> output:#SARA_USB_D##0
- U$464: device output:#3#3V#0 -> output:#SARA_USB_DET#0
- U$466: device output:#VCCIO#0 -> output:#VIN#0
- U$468: device output:#1#8V#0 -> output:#3#3V#0
- U$470: device output:#RST#1 -> output:#VCCIO#0
- U$472: device output:NI0 -> output:#1#8V#0
- U$473: device output:TP0 -> output:#RST#1
- U$474: device output:#USB_D##0 -> output:#MEAS#2
- U$476: device output:#V_USB#0 -> output:TP0
- U$478: device output:M0 -> output:#USB_D##0
- U$479: device output:CHARGE0 -> output:#V_USB#0
- U$480: device output:ASSET_TRACKER0 -> output:AG0
- U$481: device output:MIC0 -> output:M0
- U$482: device output:#EN#0 -> output:CHARGE0
- U$483: device output:#SARA_I�C#0 -> output:ASSET_TRACKER0
- U$485: device output:LTE0 -> output:#EN#0
- U$487: device output:GNSS0 -> output:#SARA_I�C#0
- U$489: device output:#SARA_INT#0 -> output:LTE0
- U$491: device output:#DSR#0 -> output:GNSS0
- U$492: device output:#SD_#CS##0 -> output:#SARA_INT#0
- U$493: device output:#IMU_PWR#0 -> output:#RI#0
- U$494: device output:#LTE_PWR#0 -> output:#DSR#0
- U$495: device output:#SD_PWR#0 -> output:#SD_#CS##0
- U$496: device output:#SARA_SCL#0 -> output:#IMU_PWR#0
- U$497: device output:#SARA_SDA#0 -> output:#LTE_PWR#0
- U$498: device output:#CIPO#0 -> output:#SD_PWR#0
- U$499: device output:22220 -> output:#SARA_SCL#0
- U$500: device output:SARA_ON0 -> output:#SARA_SDA#0
- U$501: device output:ON0 -> output:#CIPO#0
- U$502: device output:#PDM_CLK#0 -> output:22220
- U$503: device output:#PDM_DAT#0 -> output:SARA_ON0
- U$504: device output:#DSR#0 -> output:ON0
- U$505: device output:#G0#0 -> output:#PDM_CLK#0
- U$506: device output:#G1#0 -> output:#PDM_DAT#0
- U$507: device output:#G2#0 -> output:#DSR#0
- U$508: device output:#G3#0 -> output:#G0#0
- U$509: device output:#G4#0 -> output:#G1#0
- U$510: device output:#G7#0 -> output:#G2#0
- U$511: device output:#G6#0 -> output:#G3#0
- U$512: device output:#G5#0 -> output:#G4#0
- U$513: device output:#D0#1 -> output:#G7#0
- U$515: device output:NANO0 -> output:#G5#0
- U$517: value MAX17048 -> (none); device SparkFun-IC-Power:DFN-8 -> output:#D0#1
- U$518: device output:#VIN#3#0 -> output:NANO0
- U$519: device output:#ICM_INT#0 -> output:SIM0
- U$520: device output:#SARA_#ON##0 -> output:#VIN#3#0
- U10: value 1.8V/100mA -> 9DoF IMU; device SparkFun-IC-Power:SC70 -> SparkFun-Sensors:QFN24-3X3-ICM-20948
- U11: value MCP73831 -> 1.8V/100mA; device SparkFun-IC-Power:SOT23-5 -> SparkFun-IC-Power:SC70
- U12: value 3.3V -> MCP73831
- U15: value PCA9306 -> 3.3V; device SparkFun-IC-Comms:VSSOP_8PIN -> SparkFun-IC-Power:SOT23-5
- U16: value 74HC1G04 -> PCA9306; device SparkFun-IC-Logic:SOT353 -> SparkFun-IC-Comms:VSSOP_8PIN
- U17: value AP7361C-33FGE -> 74HC1G04; device SparkFun-IC-Power:UDFN-8 -> SparkFun-IC-Logic:SOT353
- U18: value SARA-R5 -> MAX17048; device SARA_R5:SARA-LGA -> SparkFun-IC-Power:DFN-8
- U19: value 9DoF IMU -> AP7361C-33FGE; device SparkFun-Sensors:QFN24-3X3-ICM-20948 -> SparkFun-IC-Power:UDFN-8
- U20: value 1.8V/100mA -> SARA-R5; device SparkFun-IC-Power:SC70 -> SARA_R5:SARA-LGA
- U21: value MCP73831 -> 9DoF IMU; device SparkFun-IC-Power:SOT23-5 -> SparkFun-Sensors:QFN24-3X3-ICM-20948
- U22: value 3.3V -> 1.8V/100mA; device SparkFun-IC-Power:SOT23-5 -> SparkFun-IC-Power:SC70
- U23: value PCA9306 -> MCP73831; device SparkFun-IC-Comms:VSSOP_8PIN -> SparkFun-IC-Power:SOT23-5
- U24: value 74HC1G04 -> 3.3V; device SparkFun-IC-Logic:SOT353 -> SparkFun-IC-Power:SOT23-5
- U25: value AP7361C-33FGE -> PCA9306; device SparkFun-IC-Power:UDFN-8 -> SparkFun-IC-Comms:VSSOP_8PIN
- U26: value SARA-R5 -> 74HC1G04; device SARA_R5:SARA-LGA -> SparkFun-IC-Logic:SOT353
- U27: value 9DoF IMU -> MAX17048; device SparkFun-Sensors:QFN24-3X3-ICM-20948 -> SparkFun-IC-Power:DFN-8
- U28: value 1.8V/100mA -> AP7361C-33FGE; device SparkFun-IC-Power:SC70 -> SparkFun-IC-Power:UDFN-8
- U29: value MCP73831 -> SARA-R5; device SparkFun-IC-Power:SOT23-5 -> SARA_R5:SARA-LGA
- U30: value 3.3V -> 9DoF IMU; device SparkFun-IC-Power:SOT23-5 -> SparkFun-Sensors:QFN24-3X3-ICM-20948
- U31: value PCA9306 -> 1.8V/100mA; device SparkFun-IC-Comms:VSSOP_8PIN -> SparkFun-IC-Power:SC70
- U32: value 74HC1G04 -> MCP73831; device SparkFun-IC-Logic:SOT353 -> SparkFun-IC-Power:SOT23-5
- U4: value AP7361C-33FGE -> MAX17048; device SparkFun-IC-Power:UDFN-8 -> SparkFun-IC-Power:DFN-8
- U6: value SARA-R5 -> AP7361C-33FGE; device SARA_R5:SARA-LGA -> SparkFun-IC-Power:UDFN-8
- U9: value 9DoF IMU -> SARA-R5; device SparkFun-Sensors:QFN24-3X3-ICM-20948 -> SARA_R5:SARA-LGA
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Connections:
- removed net N$101 (its old number): D28.C, R100.1, U17.5, VE2.2
- removed net N$102 (its old number): JP40.3, R104.2
- removed net N$109 (its old number): C85.1, C86.1, R111.1, U22.5
- removed net N$110 (its old number): C87.1, FB3.1, R111.2, TP70.P$1
- removed net N$114 (its old number): R115.1, U24.4
- removed net N$115 (its old number): JP44.1, R109.2
- removed net N$123 (its old number): R123.2, U18.13
- removed net N$124 (its old number): R124.2, U18.12
- removed net N$129 (its old number): J44.50, JP55.1
- removed net N$133 (its old number): J44.16, JP57.2
- removed net N$139 (its old number): JP58.3, R143.2
- removed net N$140 (its old number): JP58.1, R142.2
- removed net N$146 (its old number): D41.C, R146.1, U25.5, VE3.2
- removed net N$147 (its old number): JP59.3, R150.2
- removed net N$148 (its old number): JP59.1, R149.2
- removed net N$154 (its old number): C115.1, C116.1, R157.1, U30.5
- removed net N$155 (its old number): C117.1, FB4.1, R157.2, TP94.P$1
- removed net N$156 (its old number): R159.1, U31.P7, U31.P8
- removed net N$160 (its old number): JP63.1, R155.2
- removed net N$161 (its old number): R164.2, U26.4
- removed net N$168 (its old number): R169.2, U26.13
- removed net N$169 (its old number): R170.2, U26.12
- removed net N$170 (its old number): J62.53, JP64.2
- removed net N$178 (its old number): J62.16, JP76.2
- removed net N$44 (its old number): BT2.+, D9.A, R49.1, TP48.P$1
- removed net N$56 (its old number): D15.C, R54.1, U4.5, VE1.2
- removed net N$64 (its old number): C55.1, C56.1, R65.1, U12.5
- removed net N$69 (its old number): R69.1, U16.4
- removed net N$78 (its old number): R77.2, U6.13
- removed net N$83 (its old number): J26.52, JP37.1
- removed net N$88 (its old number): J26.16, JP38.2
- removed net N$93 (its old number): BT3.+, D27.A, R95.1, TP72.P$1
- removed net N$94 (its old number): JP39.3, R97.2
- removed net SARA_INT_1.8V: Q5.2, R29.1, TP11.P$1, U1.33
- removed net SARA_INT_1.8V1: Q14.2, R70.1, TP35.P$1, U6.33
- removed net SARA_INT_1.8V2: Q24.2, R116.1, TP59.P$1, U18.33
- removed net SARA_INT_1.8V3: Q34.2, R162.1, TP83.P$1, U26.33
- new net N$106: C70.1, U21.10
- new net N$107: R107.2, U23.5
- new net N$112: C87.1, FB3.1, R111.2, TP67.P$1
- new net N$113: R113.1, U25.P7, U25.P8
- new net N$117: JP46.1, R109.2
- new net N$118: R118.2, U20.4
- new net N$127: J44.53, JP47.2
- new net N$130: J44.52, JP58.1
- new net N$131: J44.50, JP57.1
- new net N$135: J44.16, JP59.2
- new net N$141: BT4.+, D40.A, R141.1, TP92.P$1
- new net N$142: JP61.3, R143.2
- new net N$143: JP61.1, R142.2
- new net N$151: JP62.1, R149.2
- new net N$152: C100.1, U30.10
- new net N$153: R153.2, U32.5
- new net N$157: C115.1, C116.1, R157.1, U33.5
- new net N$158: C117.1, FB4.1, R157.2, TP90.P$1
- new net N$162: R161.1, U35.4
- new net N$163: JP66.1, R155.2
- new net N$164: R164.2, U29.4
- new net N$172: R170.2, U29.12
- new net N$176: J62.52, JP78.1
- new net N$177: J62.50, JP77.1
- new net N$181: J62.16, JP79.2
- new net N$184: JP80.2, Q34.2, R162.1
- new net N$43: JP19.2, Q5.2, R29.1
- new net N$48: JP21.1, R50.2
- new net N$61: R61.2, U12.5
- new net N$67: R67.1, U16.P7, U16.P8
- new net N$72: R72.2, U9.4
- new net N$82: J26.51, JP28.2
- new net N$85: J26.50, JP37.1
- new net N$89: J26.16, JP39.2
- new net N$92: JP40.2, Q14.2, R70.1
- new net N$96: JP41.3, R97.2
- new net N$97: JP41.1, R96.2
- new net SARA_EXT_INT: JP19.3, U1.33
- new net SARA_EXT_INT1: JP40.3, U9.33
- new net SARA_EXT_INT2: JP60.3, U20.33
- new net SARA_EXT_INT3: JP80.3, U29.33
- new net SARA_GPIO1: JP40.1, U9.24
- new net SARA_GPIO2: JP60.1, U20.24
- new net SARA_GPIO3: JP19.1, U1.24
- new net SARA_GPIO4: JP80.1, U29.24
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Routing:
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